File: powersupply.kicad_sch (KiCad schematic)
At the start: 19 parts, among them U1 MCP1824T-2502EOT, U2 MIC5258-1.2YM5, U9 NCP752BSN33T1G

Commit message: V2
Parts:
- D1: footprint LED_SMD:LED_0402_1005Metric -> LED_SMD:LED_0805_2012Metric
Changed lines of the file:
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@@
 			)
 		)
-		(property "Footprint" "LED_SMD:LED_0402_1005Metric"
+		(property "Footprint" "LED_SMD:LED_0805_2012Metric"
 			(at 140.97 144.78 0)
 			(effects

Commit message: V5
Parts:
- C1, C2, C3, C4, C5, C6: footprint C_0805_2012Metric -> Capacitor_SMD:C_0805_2012Metric
- R1, R2, R22, R3: footprint R_0805_2012Metric -> Resistor_SMD:R_0805_2012Metric
