File: usb_to_serial.kicad_sch (KiCad schematic)
At the start: 10 parts, among them P1 USB_C_Plug, U3 CH552E, U5 USBLC6-2SC6

Commit message: V4
Parts:
- P1: value USB_C_Plug -> USB_A; footprint mta1:U261-241N-4BS60 -> Connector_USB:USB_A_Kycon_KUSBX-AS1N-B_Horizontal

Commit message: V5
Parts:
- removed P1: USB_A, Connector_USB:USB_A_Kycon_KUSBX-AS1N-B_Horizontal, symbol Connector:USB_C_Plug
- removed R29: 5.1k, R_0805_2012Metric, symbol Device:R
- added J1: USB_A, Connector_USB:USB_A_Kycon_KUSBX-AS1N-B_Horizontal, symbol Connector:USB_A
- C13, C7: footprint C_0805_2012Metric -> Capacitor_SMD:C_0805_2012Metric
Connections:
- net +5V: now also J1.1 (VBUS)
- net GND: now also J1.4 (GND), J1.5 (Shield)
- net INT_USB_IN_D+: now also J1.3 (D+)
- net INT_USB_IN_D-: now also J1.2 (D-)
- no-connect marks 12 -> 1
